Commit message: Simulation
Sims with random object

File: Manipulation/poppy_ergo_jr_new.urdf (robot description, URDF)
Before this commit: robot poppy_ergo_jr, 9 links, 8 joints
Links:
- added link movable_hidden_tip, mass 0.1; visual box size=0.005 0.005 0.005
Joints:
- added joint t8newfixed: type continuous, parent moving_tip, child movable_hidden_tip, origin xyz=0 -0.062 0 rpy=-1.5707963267949 0 0, axis 0 -1 0
