Commit message: initial dmcontrol env running

File: ergo/urdfs/ergo/poppy_ergo.dmcontrol.urdf (robot description, URDF)
Before this commit: robot Poppy_Humanoid, 37 links, 36 joints
Links:
- added link world
- link l_fixed_tip: geometry collision box size=0.020 0.025 0.003; visual box size=.001 .001 .001
- link l_moving_tip: geometry collision box size=0.003 0.025 0.02; visual box size=.001 .001 .001
- link r_fixed_tip: geometry collision box size=0.020 0.025 0.003; visual box size=.001 .001 .001
- link r_moving_tip: geometry collision box size=0.003 0.025 0.02; visual box size=.001 .001 .001
Joints:
- added joint floating_base: type floating, parent world, child pelvis, origin xyz=0 0 .43 rpy=0 0 0
