Commit message: fixed 0 angle for wrists

File: ergo/urdfs/ergo/poppy_ergo.pybullet.urdf (robot description, URDF)
Before this commit: robot Poppy_Humanoid, 36 links, 35 joints
Joints:
- joint l_wrist_x: origin xyz=0 0.025 0 rpy=0 0 0 -> xyz=0 0.025 0 rpy=3.14159265358979 0 0
- joint r_wrist_x: origin xyz=0 0.025 0 rpy=0 0 0 -> xyz=0 0.025 0 rpy=3.14159265358979 0 0

Commit message: added get_camera_image function to environment

File: ergo/urdfs/ergo/poppy_ergo.pybullet.urdf (robot description, URDF)
Before this commit: robot Poppy_Humanoid, 36 links, 35 joints
Links:
- added link camera
Joints:
- added joint head_cam: type fixed, parent head, child camera, origin xyz=0 .075 .025 rpy=0 0 0, axis 1 0 0

Commit message: fine-tuned goal distribution

File: ergo/urdfs/ergo/poppy_ergo.pybullet.urdf (robot description, URDF)
Before this commit: robot Poppy_Humanoid, 37 links, 36 joints
Links:
- link camera: mass None -> 0.06

Commit message: added fixed joints for toes and heels

File: ergo/urdfs/ergo/poppy_ergo.pybullet.urdf (robot description, URDF)
Before this commit: robot Poppy_Humanoid, 37 links, 36 joints
Links:
- added link l_heel, mass 0.06
- added link l_toe, mass 0.06
- added link r_heel, mass 0.06
- added link r_toe, mass 0.06
Joints:
- added joint l_heel: type fixed, parent l_foot, child l_heel, origin xyz=-0.02091397 -0.03580464 -0.04469591 rpy=0 0 0
- added joint l_toe: type fixed, parent l_foot, child l_toe, origin xyz=-0.01781701 -0.03594633  0.10130183 rpy=0 0 0
- added joint r_heel: type fixed, parent r_foot, child r_heel, origin xyz=0.02091397 -0.03580464 -0.04469591 rpy=0 0 0
- added joint r_toe: type fixed, parent r_foot, child r_toe, origin xyz=0.01781701 -0.03594633  0.10130183 rpy=0 0 0

Commit message: cleaning up trajectory generation

File: ergo/urdfs/ergo/poppy_ergo.pybullet.urdf (robot description, URDF)
Before this commit: robot Poppy_Humanoid, 41 links, 40 joints
Joints:
- joint l_heel: origin xyz=-0.02091397 -0.03580464 -0.04469591 rpy=0 0 0 -> xyz=-0.0210066 -0.03570167 -0.04526183 rpy=0 0 0
- joint l_toe: origin xyz=-0.01781701 -0.03594633  0.10130183 rpy=0 0 0 -> xyz=-0.01774795 -0.03446821  0.10293077 rpy=0 0 0
- joint r_heel: origin xyz=0.02091397 -0.03580464 -0.04469591 rpy=0 0 0 -> xyz=0.0210066 -0.03570167 -0.04526183 rpy=0 0 0
- joint r_toe: origin xyz=0.01781701 -0.03594633  0.10130183 rpy=0 0 0 -> xyz=0.01774795 -0.03446821  0.10293077 rpy=0 0 0

Commit message: constrained trajectory interpolation

File: ergo/urdfs/ergo/poppy_ergo.pybullet.urdf (robot description, URDF)
Before this commit: robot Poppy_Humanoid, 41 links, 40 joints
Links:
- link l_foot: geometry collision mesh filename=meshes/l_foot_respondable.STL; visual mesh filename=meshes/l_foot_respondable.STL
- link r_foot: geometry collision mesh filename=meshes/r_foot_respondable.STL; visual mesh filename=meshes/r_foot_respondable.STL
Joints:
- joint l_heel: origin xyz=-0.0210066 -0.03570167 -0.04526183 rpy=0 0 0 -> xyz=-0.0210066 -0.035 -0.04526183 rpy=0 0 0
- joint l_toe: origin xyz=-0.01774795 -0.03446821  0.10293077 rpy=0 0 0 -> xyz=-0.01774795 -0.035  0.10293077 rpy=0 0 0
- joint r_heel: origin xyz=0.0210066 -0.03570167 -0.04526183 rpy=0 0 0 -> xyz=0.0210066 -0.035 -0.04526183 rpy=0 0 0
- joint r_toe: origin xyz=0.01774795 -0.03446821  0.10293077 rpy=0 0 0 -> xyz=0.01774795 -0.035  0.10293077 rpy=0 0 0

Commit message: knuckle joints and top-down grasp trajectories

File: ergo/urdfs/ergo/poppy_ergo.pybullet.urdf (robot description, URDF)
Before this commit: robot Poppy_Humanoid, 41 links, 40 joints
Links:
- added link l_fixed_knuckle, mass .01; collision box size=0.020 0.025 0.003; visual box size=0 0 0
- added link r_fixed_knuckle, mass .01; collision box size=0.020 0.025 0.003; visual box size=0 0 0
Joints:
- added joint l_fixed_knuckle: type fixed, parent l_fixed_tip, child l_fixed_knuckle, origin xyz=0 0.05 0 rpy=0 0 0
- added joint r_fixed_knuckle: type fixed, parent r_fixed_tip, child r_fixed_knuckle, origin xyz=0 0.05 0 rpy=0 0 0
- joint l_fixed_tip: axis (none) -> 0 0 1
- joint r_fixed_tip: axis (none) -> 0 0 1

Commit message: reasonably effective grasps in baseline learner

File: ergo/urdfs/ergo/poppy_ergo.pybullet.urdf (robot description, URDF)
Before this commit: robot Poppy_Humanoid, 43 links, 42 joints
Links:
- link l_fixed_tip: mass .01 -> 1.
- link l_moving_tip: mass .01 -> 1.
- link r_fixed_tip: mass .01 -> 1.
- link r_moving_tip: mass .01 -> 1.
