Commit message: troubleshooting physics test joint limits

File: ergo/pybullet/tasks/walking/test.urdf (robot description, URDF)
Before this commit: robot walker, 5 links, 4 joints
Joints:
- joint left_ankle: limit lower=-6.14 upper=6.14 effort=100 velocity=10.0 -> lower=-3 upper=3 effort=100 velocity=10.0; origin xyz=0 0 -1 rpy=0 0 0 -> xyz=0 0 -1.3 rpy=0 0 0
- joint left_hip: limit lower=-6.14 upper=6.14 effort=100 velocity=10.0 -> lower=-20 upper=20 effort=100 velocity=10.0
- joint right_ankle: limit lower=-6.14 upper=6.14 effort=100 velocity=10.0 -> lower=-3 upper=3 effort=100 velocity=10.0; origin xyz=0 0 -1 rpy=0 0 0 -> xyz=0 0 -1.3 rpy=0 0 0
- joint right_hip: limit lower=-6.14 upper=6.14 effort=100 velocity=10.0 -> lower=-20 upper=20 effort=100 velocity=10.0
